Commit message: fix: use file:// URI for conveyor mesh to enable Gazebo rendering
Gazebo Classic silently fails to resolve package:// URIs for meshes,
so the conveyor belt visual was missing in Gazebo (only the arm showed).
Switch to file://$(find ...) which xacro resolves to an absolute path,
matching the pattern used by piper_description arm meshes.
RViz unaffected (supports both URI schemes).

File: src/agx_arm_ros/src/agx_arm_moveit/config/conveyor_cell.urdf.xacro (robot description, xacro)
@@ -28,8 +28,9 @@
   </joint>
   <!-- ════════ 传送带结构 visual (conveyor_only.stl, 不含机械臂/电控箱) ════════ -->
+  <!-- 注意: Gazebo Classic 对 package:// URI 解析不可靠, 必须用 file://$(find ...) -->
   <link name="conveyor_structure">
     <visual name="conveyor_structure_visual">
       <geometry>
-        <mesh filename="package://agx_arm_description/agx_arm_urdf/piper/meshes/conveyor_only.stl"
+        <mesh filename="file://$(find agx_arm_description)/agx_arm_urdf/piper/meshes/conveyor_only.stl"
               scale="0.001 0.001 0.001"/>
       </geometry>
